File: hardware/pcb/game_board/game_board.kicad_pcb (KiCad board)
At the start: 2 copper layers, 210.3 x 209.8 mm, 219 parts, among them J1 Conn_01x03_Male, J2 Conn_01x08, U1 ESP32_Wroom_DevKit

Commit message: Finished PCB
Parts:
- added J1: Conn_01x02, Connector_JST:JST_EH_B2B-EH-A_1x02_P2.50mm_Vertical, B.Cu at (181.6, 227.8)
- added J4: Conn_01x03, Connector_JST:JST_EH_B3B-EH-A_1x03_P2.50mm_Vertical, B.Cu at (187.7, 219.9)
- added J5: Conn_01x03, Connector_JST:JST_EH_B3B-EH-A_1x03_P2.50mm_Vertical, B.Cu at (180.0, 219.9)
- added J6: Conn_01x03, Connector_JST:JST_EH_B3B-EH-A_1x03_P2.50mm_Vertical, B.Cu at (172.4, 219.9)
- added R73: 10k, Resistor_SMD:R_0805_2012Metric, F.Cu at (188.0, 209.3)
- added R74: 10k, Resistor_SMD:R_0805_2012Metric, F.Cu at (180.3, 209.3)
- added R75: 10k, Resistor_SMD:R_0805_2012Metric, F.Cu at (172.7, 209.3)
- added REF**: MountingHole_3.2mm_M3, MountingHole:MountingHole_3.2mm_M3, F.Cu at (171.4, 97.8)
- added REF**: MountingHole_3.2mm_M3, MountingHole:MountingHole_3.2mm_M3, F.Cu at (233.7, 39.4)
- added REF**: MountingHole_3.2mm_M3, MountingHole:MountingHole_3.2mm_M3, F.Cu at (171.4, 160.0)
- added REF**: MountingHole_3.2mm_M3, MountingHole:MountingHole_3.2mm_M3, F.Cu at (108.0, 97.8)
- added REF**: MountingHole_3.2mm_M3, MountingHole:MountingHole_3.2mm_M3, F.Cu at (53.3, 39.4)
- added REF**: MountingHole_3.2mm_M3, MountingHole:MountingHole_3.2mm_M3, F.Cu at (233.7, 218.4)
- added REF**: MountingHole_3.2mm_M3, MountingHole:MountingHole_3.2mm_M3, F.Cu at (53.3, 218.4)
- added REF**: MountingHole_3.2mm_M3, MountingHole:MountingHole_3.2mm_M3, F.Cu at (108.0, 160.0)
- moved J2 17.5 mm to (208.2, 227.8), turned to 180 degrees
- renumbered J1 to J3
Connections:
- J2 pad 1: +5V -> GND
- J2 pad 2: /MOSI -> /LED / BL
- J2 pad 3: /RST -> /CS
- J2 pad 4: /DC -> /SCK
- J2 pad 5: /SCK -> /DC
- J2 pad 6: /CS -> /RST
- J2 pad 7: /LED / BL -> /MOSI
- J2 pad 8: GND -> +5V
- U1 pad 10: unconnected-(U1-Pad10) -> /Button_3
- U1 pad 11: unconnected-(U1-Pad11) -> /Button_2
- U1 pad 12: unconnected-(U1-Pad12) -> /Button_1
Routing:
- net /Button_1: track 0.00 -> 97.5 mm, vias 0 -> 1
- net /Button_2: track 0.00 -> 89.4 mm, vias 0 -> 1
- net /Button_3: track 0.00 -> 84.0 mm, vias 0 -> 1
- net +3V3: track 85.2 -> 117.9 mm
- net +5V: track 163.0 -> 168.9 mm, vias 71 -> 74
- net /SCK: track 37.6 -> 36.3 mm
- net /MOSI: track 46.3 -> 45.0 mm
- net /LED / BL: track 11.8 -> 10.5 mm
- net /DC: track 37.6 -> 36.3 mm
- net /CS: track 37.6 -> 36.3 mm
Other:
- board text added: "Button 1"
- board text added: "Button 2"
- board text added: "Button 3"
- board text added: "IN"
