File: hardware/pcb/game_board/game_board.kicad_sch (KiCad schematic)
At the start: 3 parts, among them J1 Conn_01x03_Male, J2 Conn_01x08, U1 ESP32_Wroom_DevKit

Commit message: Finished PCB
Parts:
- added J1: Conn_01x02, Connector_JST:JST_EH_B2B-EH-A_1x02_P2.50mm_Vertical, symbol Connector_Generic:Conn_01x02
- added J4, J5, J6: Conn_01x03, Connector_JST:JST_EH_B3B-EH-A_1x03_P2.50mm_Vertical, symbol Connector_Generic:Conn_01x03
- added R73, R74, R75: 10k, Resistor_SMD:R_0805_2012Metric, symbol Device:R
- renumbered J1 to J3
Connections:
- net +3V3: now also J4.3 (Pin_3), J5.3 (Pin_3), J6.3 (Pin_3)
- net +5V: now also J2.8 (Pin_8), J1.2 (Pin_2), R73.1, R74.1, R75.1; no longer J2.1 (Pin_1)
- net CS: now also J2.3 (Pin_3); no longer J2.6 (Pin_6)
- net DC: now also J2.5 (Pin_5); no longer J2.4 (Pin_4)
- net GND: now also J2.1 (Pin_1), J1.1 (Pin_1), J4.1 (Pin_1), J5.1 (Pin_1), J6.1 (Pin_1); no longer J2.8 (Pin_8)
- net LED / BL: now also J2.2 (Pin_2); no longer J2.7 (Pin_7)
- net MOSI: now also J2.7 (Pin_7); no longer J2.2 (Pin_2)
- net RST: now also J2.6 (Pin_6); no longer J2.3 (Pin_3)
- net SCK: now also J2.4 (Pin_4); no longer J2.5 (Pin_5)
- net Button_3: now reaches U1.10 (IO26)
- net Button_3: now also J6.2 (Pin_2), R75.2
- net Button_2: now reaches U1.11 (IO27)
- net Button_2: now also J5.2 (Pin_2), R74.2
- net Button_1: now reaches U1.12 (IO14)
- net Button_1: now also J4.2 (Pin_2), R73.2
Other:
- moved on the sheet: J2, J3
