File: hardware/pcb/game_board_mini/ESP-C3.kicad_sch (KiCad schematic)
At the start: 9 parts

Commit message: [PCB] Finished ESP Schematic
Parts:
- added AE?: ANT3216LL00R2400A, symbol Device:Antenna_Chip
- added C? (x2): 10p, symbol Device:C
- added C?: 1µ, symbol Device:C
- added C? (x2): 3.3p, symbol Device:C
- added J?: USB_C_Receptacle, symbol Connector:USB_C_Receptacle
- added L?: 2.2n, symbol Device:L
- added R? (x2): 5k1, symbol Device:R
- added R?: 22, symbol Device:R
- added R?: 10k, symbol Device:R
- added R?: 470, symbol Device:R
- added SW?: SW_Push, symbol Switch:SW_Push
- added U?: USBLC6-2SC6, Package_TO_SOT_SMD:SOT-23-6, symbol Power_Protection:USBLC6-2SC6
- added Y?: Crystal_GND24, symbol Device:Crystal_GND24
- C? (x2): value C -> 100n
- L?: value L -> 2.2n
Connections:
- net +3.3V: now also R?.1
- net CHIP_EN: now also C?.1, R?.2, SW?.2
- net GND: now also AE?.1 (FEED), C?.1, C?.2, C?.2, C?.2, C?.2, J?.A1 (GND), J?.A12 (GND), J?.B1 (GND), J?.B12 (GND), R?.2, R?.2, SW?.1, U?.2 (GND), Y?.2, Y?.4
- net LNA_IN: now reaches U?.1 (LNA_IN)
- net LNA_IN: now also C?.1, L?.2
- net GPIO_5: now reaches U?.10 (MTDI)
- net GPIO_6: now reaches U?.12 (MTCK)
- net GPIO_7: now reaches U?.13 (NTDO)
- net GPIO_8: now reaches U?.14 (GPIO8)
- net GPIO_9: now reaches U?.15 (GPIO9)
- net GPIO_10: now reaches U?.16 (GPIO10)
- net GPIO_20: now reaches U?.27 (U0RXD)
- net at U?.28 (U0TXD): now also R?.1
- net at U?.29 (XTAL_N): now also C?.1, Y?.3
- net at U?.30 (XTAL_P): now also R?.2
- net GPIO_0: now reaches U?.4 (XTAL_32K_P)
- net GPIO_1: now reaches U?.5 (XTAL_32K_N)
- net GPIO_2: now reaches U?.6 (GPIO2)
- net GPIO_3: now reaches U?.8 (GPIO3)
- net GPIO_4: now reaches U?.9 (MTMS)
- net C3_USB_D+ renamed USB_D+
- net USB_D+: now also U?.1 (I/O1)
- net C3_USB_D- renamed USB_D-
- net USB_D-: now also U?.3 (I/O2)
- new net: C?.2, R?.1, Y?.1
- new net: AE?.2 (PCB_Trace), C?.1, L?.1
- new net: J?.A6 (D+), J?.B6 (D+), U?.6 (I/O1)
- new net: J?.A7 (D-), J?.B7 (D-), U?.4 (I/O2)
- new net CC1: J?.A5 (CC1), R?.1
- new net CC2: J?.B5 (CC2), R?.1
- new net GPIO_21: R?.2
- new net VBUS: J?.A4 (VBUS), J?.A9 (VBUS), J?.B4 (VBUS), J?.B9 (VBUS), U?.5 (VBUS)
- no-connect marks 0 -> 18
Other:
- note added: "Note: 499R Resistor in series has to be placed on U0TXD tu suppress 80MHz Harmonics"
- note added: "Note: These SPI-Outputs are used for an external flash and should only be used for such"
- note added: "Z=(35+j10)R"
- note added: "Z=50R"
- note removed: "TODO: Dimension PI Filter"
- moved on the sheet: C?, L?
