File: hardware/pcb/game_board_mini/game_board_mini.kicad_sch (KiCad schematic)
At the start: 0 parts

Commit message: [PCB] Started routing (LEDs almost done, ESP started)
Parts:
- added J1: Conn_01x08, Connector_JST:JST_EH_B8B-EH-A_1x08_P2.50mm_Vertical, symbol Connector_Generic:Conn_01x08
- added J2: Conn_01x03_Male, Connector_PinHeader_2.54mm:PinHeader_1x03_P2.54mm_Vertical, symbol Connector:Conn_01x03_Male
- added J3, J4, J5: Conn_01x03, Connector_JST:JST_EH_B3B-EH-A_1x03_P2.50mm_Vertical, symbol Connector_Generic:Conn_01x03
- added R73, R74, R75: 10k, Resistor_SMD:R_0805_2012Metric, symbol Device:R
Connections:
- new net +3V3: J2.1 (Pin_1), J3.3 (Pin_3), J4.3 (Pin_3), J5.3 (Pin_3)
- new net +5V: J1.8 (Pin_8), R73.1, R74.1, R75.1
- new net BL: J2.3 (Pin_3)
- new net Button_1: J3.2 (Pin_2), R73.2
- new net Button_2: J4.2 (Pin_2), R74.2
- new net Button_3: J5.2 (Pin_2), R75.2
- new net CS: J1.3 (Pin_3)
- new net DC: J1.5 (Pin_5)
- new net GND: J1.1 (Pin_1), J3.1 (Pin_1), J4.1 (Pin_1), J5.1 (Pin_1)
- new net LED / BL: J1.2 (Pin_2), J2.2 (Pin_2)
- new net MOSI: J1.7 (Pin_7)
- new net RST: J1.6 (Pin_6)
- new net SCK: J1.4 (Pin_4)
Other:
- sheet ESP-C3 ports: added GPIO_0, GPIO_1, GPIO_10, GPIO_2, GPIO_20, GPIO_21, GPIO_3, GPIO_4, GPIO_5, GPIO_6, GPIO_7, GPIO_8, GPIO_9; removed none

Commit message: [PCB] Routed ESP
Parts:
- removed J2: Conn_01x03_Male, Connector_PinHeader_2.54mm:PinHeader_1x03_P2.54mm_Vertical, symbol Connector:Conn_01x03_Male
- added JP1: SolderJumper_3_Open, Jumper:SolderJumper-3_P1.3mm_Open_Pad1.0x1.5mm, symbol Jumper:SolderJumper_3_Open
Connections:
- net +3V3: now also JP1.3 (B)
- net BL: now also JP1.1 (A)
- net LED / BL: now also JP1.2 (C)
