File: hardware/pcb/game_board_mini/Connectors.kicad_sch (KiCad schematic)
At the start: 8 parts

Commit message: [PCB] Current board
Parts:
- gave numbers to parts that had none: 8
Changed lines of the file:
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@@
   (symbol (lib_id "power:+3V3") (at 236.22 86.36 0) (unit 1)
     (in_bom yes) (on_board yes) (fields_autoplaced)
-    (property "Reference" "#PWR?" (id 0) (at 236.22 90.17 0)
+    (property "Reference" "#PWR0225" (id 0) (at 236.22 90.17 0)
       (effects (font (size 1.27 1.27)) hide)
     )
@@
   (symbol (lib_id "power:+3V3") (at 144.78 86.36 0) (unit 1)
     (in_bom yes) (on_board yes) (fields_autoplaced)
-    (property "Reference" "#PWR?" (id 0) (at 144.78 90.17 0)
+    (property "Reference" "#PWR0223" (id 0) (at 144.78 90.17 0)
       (effects (font (size 1.27 1.27)) hide)
     )
@@
   (symbol (lib_id "power:GND") (at 62.23 101.6 0) (unit 1)
     (in_bom yes) (on_board yes) (fields_autoplaced)
-    (property "Reference" "#PWR?" (id 0) (at 62.23 107.95 0)
+    (property "Reference" "#PWR0218" (id 0) (at 62.23 107.95 0)
       (effects (font (size 1.27 1.27)) hide)
     )
@@
   (symbol (lib_id "power:+3V3") (at 195.58 86.36 0) (unit 1)
     (in_bom yes) (on_board yes) (fields_autoplaced)
-    (property "Reference" "#PWR?" (id 0) (at 195.58 90.17 0)
+    (property "Reference" "#PWR0228" (id 0) (at 195.58 90.17 0)
       (effects (font (size 1.27 1.27)) hide)
     )
@@
   (symbol (lib_id "power:GND") (at 193.04 101.6 0) (unit 1)
     (in_bom yes) (on_board yes) (fields_autoplaced)
-    (property "Reference" "#PWR?" (id 0) (at 193.04 107.95 0)
+    (property "Reference" "#PWR0222" (id 0) (at 193.04 107.95 0)
       (effects (font (size 1.27 1.27)) hide)
     )
@@
   (symbol (lib_id "Device:R") (at 135.89 91.44 0) (unit 1)
     (in_bom yes) (on_board yes) (fields_autoplaced)
-    (property "Reference" "R?" (id 0) (at 138.43 90.1699 0)
+    (property "Reference" "R73" (id 0) (at 138.43 90.1699 0)
       (effects (font (size 1.27 1.27)) (justify left))
     )
@@
   (symbol (lib_id "Connector_Generic:Conn_01x03") (at 201.93 96.52 0) (mirror x) (unit 1)
     (in_bom yes) (on_board yes) (fields_autoplaced)
-    (property "Reference" "J?" (id 0) (at 201.93 87.63 0))
+    (property "Reference" "J4" (id 0) (at 201.93 87.63 0))
     (property "Value" "Conn_01x03" (id 1) (at 201.93 90.17 0))
     (property "Footprint" "Connector_JST:JST_PH_B3B-PH-K_1x03_P2.00mm_Vertical" (id 2) (at 201.93 96.52 0)
@@
   (symbol (lib_id "Connector_Generic:Conn_01x03") (at 151.13 96.52 0) (mirror x) (unit 1)
     (in_bom yes) (on_board yes) (fields_autoplaced)
-    (property "Reference" "J?" (id 0) (at 151.13 87.63 0))
+    (property "Reference" "J3" (id 0) (at 151.13 87.63 0))
     (property "Value" "Conn_01x03" (id 1) (at 151.13 90.17 0))
     (property "Footprint" "Connector_JST:JST_PH_B3B-PH-K_1x03_P2.00mm_Vertical" (id 2) (at 151.13 96.52 0)
@@
   (symbol (lib_id "power:GND") (at 142.24 101.6 0) (unit 1)
     (in_bom yes) (on_board yes) (fields_autoplaced)
-    (property "Reference" "#PWR?" (id 0) (at 142.24 107.95 0)
+    (property "Reference" "#PWR0221" (id 0) (at 142.24 107.95 0)
       (effects (font (size 1.27 1.27)) hide)
     )
@@
   (symbol (lib_id "power:+3V3") (at 62.23 118.11 0) (unit 1)
     (in_bom yes) (on_board yes) (fields_autoplaced)
-    (property "Reference" "#PWR?" (id 0) (at 62.23 121.92 0)
+    (property "Reference" "#PWR0217" (id 0) (at 62.23 121.92 0)
       (effects (font (size 1.27 1.27)) hide)
     )
@@
   (symbol (lib_id "power:+3V3") (at 245.11 86.36 0) (unit 1)
     (in_bom yes) (on_board yes) (fields_autoplaced)
-    (property "Reference" "#PWR?" (id 0) (at 245.11 90.17 0)
+    (property "Reference" "#PWR0226" (id 0) (at 245.11 90.17 0)
       (effects (font (size 1.27 1.27)) hide)
     )
@@
   (symbol (lib_id "Jumper:SolderJumper_3_Open") (at 62.23 124.46 90) (unit 1)
     (in_bom yes) (on_board yes) (fields_autoplaced)
-    (property "Reference" "JP?" (id 0) (at 59.69 123.1899 90)
+    (property "Reference" "JP1" (id 0) (at 59.69 123.1899 90)
       (effects (font (size 1.27 1.27)) (justify left))
     )
@@
   (symbol (lib_id "power:+3V3") (at 186.69 86.36 0) (unit 1)
     (in_bom yes) (on_board yes) (fields_autoplaced)
-    (property "Reference" "#PWR?" (id 0) (at 186.69 90.17 0)
+    (property "Reference" "#PWR0227" (id 0) (at 186.69 90.17 0)
       (effects (font (size 1.27 1.27)) hide)
     )
@@
   (symbol (lib_id "Connector_Generic:Conn_01x03") (at 251.46 96.52 0) (mirror x) (unit 1)
     (in_bom yes) (on_board yes) (fields_autoplaced)
-    (property "Reference" "J?" (id 0) (at 251.46 87.63 0))
+    (property "Reference" "J5" (id 0) (at 251.46 87.63 0))
     (property "Value" "Conn_01x03" (id 1) (at 251.46 90.17 0))
     (property "Footprint" "Connector_JST:JST_PH_B3B-PH-K_1x03_P2.00mm_Vertical" (id 2) (at 251.46 96.52 0)
@@
   (symbol (lib_id "power:GND") (at 242.57 101.6 0) (unit 1)
     (in_bom yes) (on_board yes) (fields_autoplaced)
-    (property "Reference" "#PWR?" (id 0) (at 242.57 107.95 0)
+    (property "Reference" "#PWR0220" (id 0) (at 242.57 107.95 0)
       (effects (font (size 1.27 1.27)) hide)
     )
@@
   (symbol (lib_id "Device:R") (at 186.69 91.44 0) (unit 1)
     (in_bom yes) (on_board yes) (fields_autoplaced)
-    (property "Reference" "R?" (id 0) (at 189.23 90.1699 0)
+    (property "Reference" "R74" (id 0) (at 189.23 90.1699 0)
       (effects (font (size 1.27 1.27)) (justify left))
     )
@@
   (symbol (lib_id "Connector_Generic:Conn_01x08") (at 71.12 92.71 0) (mirror x) (unit 1)
     (in_bom yes) (on_board yes) (fields_autoplaced)
-    (property "Reference" "J?" (id 0) (at 71.12 76.2 0))
+    (property "Reference" "J1" (id 0) (at 71.12 76.2 0))
     (property "Value" "Conn_01x08" (id 1) (at 71.12 78.74 0))
     (property "Footprint" "Connector_JST:JST_PH_B8B-PH-K_1x08_P2.00mm_Vertical" (id 2) (at 71.12 92.71 0)
@@
   (symbol (lib_id "power:+5V") (at 62.23 63.5 0) (unit 1)
     (in_bom yes) (on_board yes) (fields_autoplaced)
-    (property "Reference" "#PWR?" (id 0) (at 62.23 67.31 0)
+    (property "Reference" "#PWR0219" (id 0) (at 62.23 67.31 0)
       (effects (font (size 1.27 1.27)) hide)
     )
@@
   (symbol (lib_id "power:+3V3") (at 135.89 86.36 0) (unit 1)
     (in_bom yes) (on_board yes) (fields_autoplaced)
-    (property "Reference" "#PWR?" (id 0) (at 135.89 90.17 0)
+    (property "Reference" "#PWR0224" (id 0) (at 135.89 90.17 0)
       (effects (font (size 1.27 1.27)) hide)
     )
@@
   (symbol (lib_id "Device:R") (at 236.22 91.44 0) (unit 1)
     (in_bom yes) (on_board yes) (fields_autoplaced)
-    (property "Reference" "R?" (id 0) (at 238.76 90.1699 0)
-      (effects (font (size 1.27 1.27)) (justify left))
-    )
+    (property "Reference" "R75" (id 0) (at 238.76 90.1699 0)
+      (effects (font (size 1.27 1.27)) (justify left))
+    )
